Commit message: added modules and pallet

File: omtp_support/urdf/omtp_factory.xacro (robot description, xacro)
@@ -37,5 +37,5 @@
   <xacro:include filename="$(find omtp_support)/urdf/robot_pedestal/robot_pedestal.urdf.xacro"/>
   <xacro:robot_pedestal_urdf pedestal_prefix="robot1_" pedestal_parent="world_interface" pedestal_height="0.95">
-    <origin xyz="-1.5 1.5 0.0" rpy="0 0 0"/>
+    <origin xyz="-1 7.3 0.0" rpy="0 0 0"/>
   </xacro:robot_pedestal_urdf>
   <!-- ==================================================== -->
@@ -44,44 +44,52 @@
   <xacro:include filename="$(find omtp_support)/urdf/robot_pedestal/robot_pedestal.urdf.xacro"/>
   <xacro:robot_pedestal_urdf pedestal_prefix="robot2_" pedestal_parent="world_interface" pedestal_height="0.95">
-    <origin xyz="-2.8 -1.5 0.0" rpy="0 0 0"/>
+    <origin xyz="-1 2.5 0.0" rpy="0 0 0"/>
   </xacro:robot_pedestal_urdf>
- <!-- ==================================================== -->
-  <!-- Bins -->
   <!-- ==================================================== -->
-  <xacro:include filename="$(find omtp_support)/urdf/bin/bin.urdf.xacro"/>
-  <xacro:bin_urdf prefix="bin_1"/>
-  <xacro:bin_urdf prefix="bin_2"/>
-  <xacro:bin_urdf prefix="bin_3"/>
-  <xacro:bin_urdf prefix="bin_4"/>
-  <xacro:bin_urdf prefix="bin_5"/>
-  <!-- Bin 1 -->
-  <joint name="bin_1_joint" type="fixed">
-    <parent link="world_interface" />
-    <child link="bin_1_base_link" />
-    <origin xyz="-0.3 1.2 0.0" rpy="0 0 0" />
-  </joint>
-  <!-- Bin 2 -->
-  <joint name="bin_2_joint" type="fixed">
-    <parent link="world_interface" />
-    <child link="bin_2_base_link" />
-    <origin xyz="-0.3 0.4 0.0" rpy="0 0 0" />
-  </joint>
-  <!-- Bin 3 -->
-  <joint name="bin_3_joint" type="fixed">
-    <parent link="world_interface" />
-    <child link="bin_3_base_link" />
-    <origin xyz="-0.3 -0.4 0.0" rpy="0 0 0" />
-  </joint>
-  <!-- Bin 4 -->
-  <joint name="bin_4_joint" type="fixed">
-    <parent link="world_interface" />
-    <child link="bin_4_base_link" />
-    <origin xyz="-0.3 -1.2 0.0" rpy="0 0 0" />
-  </joint>
-  <!-- Bin 5 -->
-  <joint name="bin_5_joint" type="fixed">
-    <parent link="world_interface" />
-    <child link="bin_5_base_link" />
-    <origin xyz="-0.3 -2.0 0.0" rpy="0 0 0" />
-  </joint>
+  <!-- module -->
+  <!-- ==================================================== -->
+  <!-- module 1 -->
+  <xacro:include filename="$(find aau_lab_ros_models)/urdf/festo_straight_module/festo_straight_module.urdf.xacro"/>
+  <xacro:festo_module_urdf module_prefix = "module1_" festo_module_parent="world_interface">
+    <origin xyz="-0.3 7.4 0.0" rpy="0 0 0" />
+  </xacro:festo_module_urdf>
+  <!-- module 2 -->
+  <xacro:include filename="$(find aau_lab_ros_models)/urdf/festo_straight_module/festo_straight_module.urdf.xacro"/>
+  <xacro:festo_module_urdf module_prefix = "module2_" festo_module_parent="world_interface">
+    <origin xyz="-0.3 6.2 0.0" rpy="0 0 0" />
+  </xacro:festo_module_urdf>
+   <!-- module 3 -->
+  <xacro:include filename="$(find aau_lab_ros_models)/urdf/festo_robot_module/festo_robot_module.urdf.xacro"/>
+  <xacro:festo_robot_module_urdf module_prefix = "module3_" festo_module_parent="world_interface" >
+   <origin xyz="-0.3 5.0 0.0" rpy="0 0 0" />
+  </xacro:festo_robot_module_urdf>
+ <!-- module 4 -->
+  <xacro:include filename="$(find aau_lab_ros_models)/urdf/festo_t_module/festo_t_module.urdf.xacro"/>
+  <xacro:festo_t_module_urdf module_prefix = "module4_" festo_module_parent="world_interface">
+   <origin xyz="-0.3 3.8 0.0" rpy="0 0 0" />
+  </xacro:festo_t_module_urdf>
+  <!-- module 5 -->
+  <xacro:include filename="$(find aau_lab_ros_models)/urdf/festo_straight_module/festo_straight_module.urdf.xacro"/>
+  <xacro:festo_module_urdf module_prefix = "module5_" festo_module_parent="world_interface">
+    <origin xyz="-0.3 2.6 0.0" rpy="0 0 0" />
+  </xacro:festo_module_urdf>
+  <!-- module 6 -->
+  <xacro:include filename="$(find aau_lab_ros_models)/urdf/festo_straight_module/festo_straight_module.urdf.xacro"/>
+  <xacro:festo_module_urdf module_prefix = "module6_" festo_module_parent="world_interface">
+    <origin xyz="-1.3 3.8 0.0" rpy="0 0 55" />
+  </xacro:festo_module_urdf>
+  <!-- module 7 -->
+  <xacro:include filename="$(find aau_lab_ros_models)/urdf/festo_bypass_module/festo_bypass_module.urdf.xacro"/>
+  <xacro:festo_bypass_module_urdf module_prefix = "module7_" festo_module_parent="world_interface">
+    <origin xyz="-2.5 3.8 0.0" rpy="0 0 1.6" />
+  </xacro:festo_bypass_module_urdf>
+  <!-- ==================================================== -->
+  <!-- objects -->
+  <!-- ==================================================== -->
+<!-- pallet -->
+  <xacro:include filename="$(find aau_lab_ros_models)/urdf/eu_pallet/eu_pallet.urdf.xacro"/>
+  <xacro:eu_pallet_urdf eu_pallet_prefix = "pallet1_" eu_pallet_parent="world_interface">
+    <origin xyz="1.5 3.8 0.0" rpy="0 0 0" />
+  </xacro:eu_pallet_urdf>
+<!-- box -->
 </robot>
