Commit message: removed repetitions in urdf file

File: src/omtp_lecture_1/omtp_support/urdf/omtp_factory.xacro (robot description, xacro)
@@ -1209,189 +1209,4 @@
         <child link="n1__nurse" />
     </joint>
-<transmission name="trans_panda_1_joint1">
-        <type>transmission_interface/SimpleTransmission</type>
-        <joint name="panda_1_joint1">
-            <hardwareInterface>hardware_interface/EffortJointInterface</hardwareInterface>
-        </joint>
-        <actuator name="panda_1_joint1_motor">
-            <hardwareInterface>hardware_interface/EffortJointInterface</hardwareInterface>
-            <mechanicalReduction>1</mechanicalReduction>
-        </actuator>
-    </transmission>
-    <transmission name="trans_panda_1_joint2">
-        <type>transmission_interface/SimpleTransmission</type>
-        <joint name="panda_1_joint2">
-            <hardwareInterface>hardware_interface/EffortJointInterface</hardwareInterface>
-        </joint>
-        <actuator name="panda_1_joint2_motor">
-            <hardwareInterface>hardware_interface/EffortJointInterface</hardwareInterface>
-            <mechanicalReduction>1</mechanicalReduction>
-        </actuator>
-    </transmission>
-    <transmission name="trans_panda_1_joint3">
-        <type>transmission_interface/SimpleTransmission</type>
-        <joint name="panda_1_joint3">
-            <hardwareInterface>hardware_interface/EffortJointInterface</hardwareInterface>
-        </joint>
-        <actuator name="panda_1_joint3_motor">
-            <hardwareInterface>hardware_interface/EffortJointInterface</hardwareInterface>
-            <mechanicalReduction>1</mechanicalReduction>
-        </actuator>
-    </transmission>
-    <transmission name="trans_panda_1_joint4">
-        <type>transmission_interface/SimpleTransmission</type>
-        <joint name="panda_1_joint4">
-            <hardwareInterface>hardware_interface/EffortJointInterface</hardwareInterface>
-        </joint>
-        <actuator name="panda_1_joint4_motor">
-            <hardwareInterface>hardware_interface/EffortJointInterface</hardwareInterface>
-            <mechanicalReduction>1</mechanicalReduction>
-        </actuator>
-    </transmission>
-    <transmission name="trans_panda_1_joint5">
-        <type>transmission_interface/SimpleTransmission</type>
-        <joint name="panda_1_joint5">
-            <hardwareInterface>hardware_interface/EffortJointInterface</hardwareInterface>
-        </joint>
-        <actuator name="panda_1_joint5_motor">
-            <hardwareInterface>hardware_interface/EffortJointInterface</hardwareInterface>
-            <mechanicalReduction>1</mechanicalReduction>
-        </actuator>
-    </transmission>
-    <transmission name="trans_panda_1_joint6">
-        <type>transmission_interface/SimpleTransmission</type>
-        <joint name="panda_1_joint6">
-            <hardwareInterface>hardware_interface/EffortJointInterface</hardwareInterface>
-        </joint>
-        <actuator name="panda_1_joint6_motor">
-            <hardwareInterface>hardware_interface/EffortJointInterface</hardwareInterface>
-            <mechanicalReduction>1</mechanicalReduction>
-        </actuator>
-    </transmission>
-    <transmission name="trans_panda_1_joint7">
-        <type>transmission_interface/SimpleTransmission</type>
-        <joint name="panda_1_joint7">
-            <hardwareInterface>hardware_interface/EffortJointInterface</hardwareInterface>
-        </joint>
-        <actuator name="panda_1_joint7_motor">
-            <hardwareInterface>hardware_interface/EffortJointInterface</hardwareInterface>
-            <mechanicalReduction>1</mechanicalReduction>
-        </actuator>
-    </transmission>
-    <transmission name="trans_panda_1_finger_joint1">
-        <type>transmission_interface/SimpleTransmission</type>
-        <joint name="panda_1_finger_joint1">
-            <hardwareInterface>hardware_interface/EffortJointInterface</hardwareInterface>
-        </joint>
-        <actuator name="panda_1_finger_joint1_motor">
-            <hardwareInterface>hardware_interface/EffortJointInterface</hardwareInterface>
-            <mechanicalReduction>1</mechanicalReduction>
-        </actuator>
-    </transmission>
-    <transmission name="trans_panda_1_finger_joint2">
-        <type>transmission_interface/SimpleTransmission</type>
-        <joint name="panda_1_finger_joint2">
-            <hardwareInterface>hardware_interface/EffortJointInterface</hardwareInterface>
-        </joint>
-        <actuator name="panda_1_finger_joint2_motor">
-            <hardwareInterface>hardware_interface/EffortJointInterface</hardwareInterface>
-            <mechanicalReduction>1</mechanicalReduction>
-        </actuator>
-    </transmission>
-    <transmission name="trans_panda_2_joint1">
-        <type>transmission_interface/SimpleTransmission</type>
-        <joint name="panda_2_joint1">
-            <hardwareInterface>hardware_interface/EffortJointInterface</hardwareInterface>
-        </joint>
-        <actuator name="panda_2_joint1_motor">
-            <hardwareInterface>hardware_interface/EffortJointInterface</hardwareInterface>
-            <mechanicalReduction>1</mechanicalReduction>
-        </actuator>
-    </transmission>
-    <transmission name="trans_panda_2_joint2">
-        <type>transmission_interface/SimpleTransmission</type>
-        <joint name="panda_2_joint2">
-            <hardwareInterface>hardware_interface/EffortJointInterface</hardwareInterface>
-        </joint>
-        <actuator name="panda_2_joint2_motor">
-            <hardwareInterface>hardware_interface/EffortJointInterface</hardwareInterface>
-            <mechanicalReduction>1</mechanicalReduction>
-        </actuator>
-    </transmission>
-    <transmission name="trans_panda_2_joint3">
-        <type>transmission_interface/SimpleTransmission</type>
-        <joint name="panda_2_joint3">
-            <hardwareInterface>hardware_interface/EffortJointInterface</hardwareInterface>
-        </joint>
-        <actuator name="panda_2_joint3_motor">
-            <hardwareInterface>hardware_interface/EffortJointInterface</hardwareInterface>
-            <mechanicalReduction>1</mechanicalReduction>
-        </actuator>
-    </transmission>
-    <transmission name="trans_panda_2_joint4">
-        <type>transmission_interface/SimpleTransmission</type>
-        <joint name="panda_2_joint4">
-            <hardwareInterface>hardware_interface/EffortJointInterface</hardwareInterface>
-        </joint>
-        <actuator name="panda_2_joint4_motor">
-            <hardwareInterface>hardware_interface/EffortJointInterface</hardwareInterface>
-            <mechanicalReduction>1</mechanicalReduction>
-        </actuator>
-    </transmission>
-    <transmission name="trans_panda_2_joint5">
-        <type>transmission_interface/SimpleTransmission</type>
-        <joint name="panda_2_joint5">
-            <hardwareInterface>hardware_interface/EffortJointInterface</hardwareInterface>
-        </joint>
-        <actuator name="panda_2_joint5_motor">
-            <hardwareInterface>hardware_interface/EffortJointInterface</hardwareInterface>
-            <mechanicalReduction>1</mechanicalReduction>
-        </actuator>
-    </transmission>
-    <transmission name="trans_panda_2_joint6">
-        <type>transmission_interface/SimpleTransmission</type>
-        <joint name="panda_2_joint6">
-            <hardwareInterface>hardware_interface/EffortJointInterface</hardwareInterface>
-        </joint>
-        <actuator name="panda_2_joint6_motor">
-            <hardwareInterface>hardware_interface/EffortJointInterface</hardwareInterface>
-            <mechanicalReduction>1</mechanicalReduction>
-        </actuator>
-    </transmission>
-    <transmission name="trans_panda_2_joint7">
-        <type>transmission_interface/SimpleTransmission</type>
-        <joint name="panda_2_joint7">
-            <hardwareInterface>hardware_interface/EffortJointInterface</hardwareInterface>
-        </joint>
-        <actuator name="panda_2_joint7_motor">
-            <hardwareInterface>hardware_interface/EffortJointInterface</hardwareInterface>
-            <mechanicalReduction>1</mechanicalReduction>
-        </actuator>
-    </transmission>
-    <transmission name="trans_panda_2_finger_joint1">
-        <type>transmission_interface/SimpleTransmission</type>
-        <joint name="panda_2_finger_joint1">
-            <hardwareInterface>hardware_interface/EffortJointInterface</hardwareInterface>
-        </joint>
-        <actuator name="panda_2_finger_joint1_motor">
-            <hardwareInterface>hardware_interface/EffortJointInterface</hardwareInterface>
-            <mechanicalReduction>1</mechanicalReduction>
-        </actuator>
-    </transmission>
-    <transmission name="trans_panda_2_finger_joint2">
-        <type>transmission_interface/SimpleTransmission</type>
-        <joint name="panda_2_finger_joint2">
-            <hardwareInterface>hardware_interface/EffortJointInterface</hardwareInterface>
-        </joint>
-        <actuator name="panda_2_finger_joint2_motor">
-            <hardwareInterface>hardware_interface/EffortJointInterface</hardwareInterface>
-            <mechanicalReduction>1</mechanicalReduction>
-        </actuator>
-    </transmission>
-    <gazebo>
-        <plugin filename="libgazebo_ros_control.so" name="gazebo_ros_control">
-            <robotNamespace>/</robotNamespace>
-        </plugin>
-    </gazebo>
     <transmission name="trans_panda_1_joint1">
         <type>transmission_interface/SimpleTransmission</type>

Commit message: made object to manipulate

File: src/omtp_lecture_1/omtp_support/urdf/omtp_factory.xacro (robot description, xacro)
@@ -33,5 +33,5 @@
             </geometry>
         </collision>
-<inertial>
+        <inertial>
             <inertia ixx="1.0" ixy="0" ixz="0" iyy="1.0" iyz="0" izz="1.0" />
             <mass value="100" />
