Commit message: fixed fatal error and add stuff

File: src/omtp_course_files_lecture_1_2022/omtp_course_files_lecture_1_2022/omtp_support/urdf/omtp.urdf (robot description, URDF)
Before this commit: robot omtp, 37 links, 36 joints
Links:
- added link n1__nurse, mass 25; collision mesh filename=package://aau_lab_ros_models/meshes/nurse/nurse.dae; visual mesh filename=package://aau_lab_ros_models/meshes/nurse/nurse.dae
- link panda_1_leftfinger: mass 0.1 -> None; geometry visual mesh filename=package://franka_description/meshes/visual/finger.dae
- link panda_1_rightfinger: mass 0.1 -> None; geometry visual mesh filename=package://franka_description/meshes/visual/finger.dae
- link panda_2_leftfinger: mass 0.1 -> None; geometry visual mesh filename=package://franka_description/meshes/visual/finger.dae
- link panda_2_rightfinger: mass 0.1 -> None; geometry visual mesh filename=package://franka_description/meshes/visual/finger.dae
Joints:
- added joint n1__to_world_interface: type fixed, parent ep1__eu_pallet, child n1__nurse, origin xyz=0.0 0.0 0.15 rpy=0 0 3.141592653589793

File: src/omtp_course_files_lecture_1_2022/omtp_course_files_lecture_1_2022/omtp_support/urdf/omtp_factory.xacro (robot description, xacro)
@@ -80,3 +80,8 @@
       <origin xyz="1.0 0.0 0.0" rpy="0 0 0"/>
   </xacro:eu_pallet_urdf>
+  <!-- example nurse model -->
+  <xacro:include filename="$(find aau_lab_ros_models)/urdf/nurse/nurse.urdf.xacro"/>
+  <xacro:nurse_urdf nurse_prefix="n1_" nurse_parent="ep1__eu_pallet">
+      <origin xyz="0.0 0.0 0.15" rpy="0 0 ${pi}"/>
+  </xacro:nurse_urdf>
 </robot>

File: src/omtp_course_files_lecture_1_2022/omtp_course_files_lecture_1_2022/omtp_support/urdf/omtp_factory_urdf.urdf.xacro (robot description, xacro)
@@ -447,13 +447,13 @@
         </visual>
         <collision>
-          <origin xyz="0 0 0" rpy="0 0 ${pi}"/>
-          <geometry>
-            <mesh filename="package://franka_description/meshes/collision/finger.stl"/>
-          </geometry>
+            <origin xyz="0 0 0" rpy="0 0 ${pi}"/>
+            <geometry>
+                <mesh filename="package://franka_description/meshes/collision/finger.stl"/>
+            </geometry>
         </collision>
         <inertial>
-          <origin xyz="0 0 0" rpy="0 0 ${pi}" />
-          <mass value="0.1" />
-          <inertia ixx="0.1" ixy="0.0" ixz="0.0" iyy="0.1" iyz="0.0" izz="0.1" />
+            <origin xyz="0 0 0" rpy="0 0 ${pi}" />
+            <mass value="0.1" />
+            <inertia ixx="0.1" ixy="0.0" ixz="0.0" iyy="0.1" iyz="0.0" izz="0.1" />
         </inertial>
     </link>
@@ -466,13 +466,13 @@
         </visual>
         <collision>
-          <origin xyz="0 0 0" rpy="0 0 ${pi}"/>
-          <geometry>
-            <mesh filename="package://franka_description/meshes/collision/finger.stl"/>
-          </geometry>
+            <origin xyz="0 0 0" rpy="0 0 ${pi}"/>
+            <geometry>
+                <mesh filename="package://franka_description/meshes/collision/finger.stl"/>
+            </geometry>
         </collision>
         <inertial>
-          <origin xyz="0 0 0" rpy="0 0 ${pi}" />
-          <mass value="0.1" />
-          <inertia ixx="0.1" ixy="0.0" ixz="0.0" iyy="0.1" iyz="0.0" izz="0.1" />
+            <origin xyz="0 0 0" rpy="0 0 ${pi}" />
+            <mass value="0.1" />
+            <inertia ixx="0.1" ixy="0.0" ixz="0.0" iyy="0.1" iyz="0.0" izz="0.1" />
         </inertial>
     </link>
@@ -899,13 +899,13 @@
         </visual>
         <collision>
-          <origin xyz="0 0 0" rpy="0 0 ${pi}"/>
-          <geometry>
-            <mesh filename="package://franka_description/meshes/collision/finger.stl"/>
-          </geometry>
+            <origin xyz="0 0 0" rpy="0 0 ${pi}"/>
+            <geometry>
+                <mesh filename="package://franka_description/meshes/collision/finger.stl"/>
+            </geometry>
         </collision>
         <inertial>
-          <origin xyz="0 0 0" rpy="0 0 ${pi}" />
-          <mass value="0.1" />
-          <inertia ixx="0.1" ixy="0.0" ixz="0.0" iyy="0.1" iyz="0.0" izz="0.1" />
+            <origin xyz="0 0 0" rpy="0 0 ${pi}" />
+            <mass value="0.1" />
+            <inertia ixx="0.1" ixy="0.0" ixz="0.0" iyy="0.1" iyz="0.0" izz="0.1" />
         </inertial>
     </link>
@@ -918,13 +918,13 @@
         </visual>
         <collision>
-          <origin xyz="0 0 0" rpy="0 0 ${pi}"/>
-          <geometry>
-            <mesh filename="package://franka_description/meshes/collision/finger.stl"/>
-          </geometry>
+            <origin xyz="0 0 0" rpy="0 0 ${pi}"/>
+            <geometry>
+                <mesh filename="package://franka_description/meshes/collision/finger.stl"/>
+            </geometry>
         </collision>
         <inertial>
-          <origin xyz="0 0 0" rpy="0 0 ${pi}" />
-          <mass value="0.1" />
-          <inertia ixx="0.1" ixy="0.0" ixz="0.0" iyy="0.1" iyz="0.0" izz="0.1" />
+            <origin xyz="0 0 0" rpy="0 0 ${pi}" />
+            <mass value="0.1" />
+            <inertia ixx="0.1" ixy="0.0" ixz="0.0" iyy="0.1" iyz="0.0" izz="0.1" />
         </inertial>
     </link>
@@ -1189,4 +1189,26 @@
         <child link="ep1__eu_pallet" />
     </joint>
+    <!-- Links -->
+    <link name="n1__nurse">
+        <visual>
+            <geometry>
+                <mesh filename="package://aau_lab_ros_models/meshes/nurse/nurse.dae" />
+            </geometry>
+        </visual>
+        <collision>
+            <geometry>
+                <mesh filename="package://aau_lab_ros_models/meshes/nurse/nurse.dae" />
+            </geometry>
+        </collision>
+<inertial>
+            <inertia ixx="1.0" ixy="0" ixz="0" iyy="1.0" iyz="0" izz="1.0" />
+            <mass value="25" />
+        </inertial>
+    </link>
+    <joint name="n1__to_world_interface" type="fixed">
+        <origin rpy="0 0 3.141592653589793" xyz="0.0 0.0 0.15" />
+        <parent link="ep1__eu_pallet" />
+        <child link="n1__nurse" />
+    </joint>
 <transmission name="trans_panda_1_joint1">
         <type>transmission_interface/SimpleTransmission</type>

File: src/omtp_course_files_lecture_8_2022/lecture5_files/omtp_lecture8/urdf/omtp_panda_2d_cam.urdf.xacro (robot description, xacro)
@@ -2,5 +2,5 @@
 <robot name="omtp"
   xmlns:xacro="http://www.ros.org/wiki/xacro">
-  <xacro:include filename="$(find omtp_support)/urdf/omtp_factory2.urdf.xacro"/>
+  <xacro:include filename="$(find omtp_support)/urdf/omtp_factory_urdf.urdf.xacro"/>
   <!-- ==================================================== -->
   <!-- 2D camera for Gazebo                                 -->

File: src/omtp_lecture3/urdf/omtp_panda.urdf.xacro (robot description, xacro)
@@ -3,5 +3,5 @@
   xmlns:xacro="http://www.ros.org/wiki/xacro">
   <!-- Insert Panda robot -->
-  <xacro:include filename="$(find omtp_support)/urdf/omtp_factory2.urdf.xacro"/>
+  <xacro:include filename="$(find omtp_support)/urdf/omtp_factory_urdf.urdf.xacro"/>
   <!-- ==================================================== -->
   <!-- 2D camera for Gazebo                                 -->
@@ -12,5 +12,5 @@
     <axis xyz="0 1 0" />
     <origin xyz="0 0 1.2" rpy="0 0 0"/>
-    <parent link="world"/>
+    <parent link="panda_1_link0"/>
     <child link="camera_link"/>
   </joint>
